File: Electronics/rhoby_motor(L6205).sch (EAGLE design)
At the start: 71 parts, among them IC1 L6205PD, IC2 L6205PD, IC3 L6205PD, IC4 74AC14D, IC5 L6205PD, IC6 74AC14D, J1 22-27-2041-04, J23 22-27-2041-04, J3 22-27-2041-04, J5 22-27-2041-04, J7 22-27-2041-04

Commit message: Changed some connectors
Parts:
- removed SV1, SV3: (no value), con-lstb:MA08-2
- removed SV2: (no value), con-lstb:MA08-1
- removed SV4: (no value), con-lstb:MA04-2
- removed SV5, SV6, SV7, SV8: (no value), con-lstb:MA06-1
- added JP11, JP12, JP13, JP14: (no value), pinhead:PINHD-1X6
- added JP15: (no value), pinhead:PINHD-2X8
- added JP16: (no value), pinhead:PINHD-2X4
- added JP17, JP18, JP19, JP20: (no value), pinhead:PINHD-2X3
Connections:
- net +5V: now also JP17.3, JP17.4, JP18.3, JP18.4, JP19.3, JP19.4, JP20.3, JP20.4; no longer SV1.1, SV1.11, SV1.13, SV1.15, SV1.3, SV1.5, SV1.7, SV1.9
- net ENC1_IN: now also JP15.1; no longer SV3.1
- net ENC2_IN: now also JP15.9; no longer SV3.9
- net ENC3_IN: now also JP15.2; no longer SV3.2
- net ENC4_IN: now also JP15.10; no longer SV3.10
- net GND: now also JP15.11, JP15.12, JP15.15, JP15.16, JP15.3, JP15.4, JP15.7, JP15.8, JP17.5, JP17.6, JP18.5, JP18.6, JP19.5, JP19.6, JP20.5, JP20.6; no longer SV1.10, SV1.12, SV1.14, SV1.16, SV1.2, SV1.4, SV1.6, SV1.8, SV3.11, SV3.12, SV3.15, SV3.16, SV3.3, SV3.4, SV3.7, SV3.8
- net HALL1: now also JP16.1; no longer SV4.1
- net HALL1_IN: now also JP17.1; no longer SV2.1
- net HALL2: now also JP16.3; no longer SV4.3
- net HALL2_IN: now also JP17.2; no longer SV2.2
- net HALL3: now also JP16.5; no longer SV4.5
- net HALL3_IN: now also JP18.1; no longer SV2.3
- net HALL4: now also JP16.7; no longer SV4.7
- net HALL4_IN: now also JP18.2; no longer SV2.4
- net HALL5: now also JP16.2; no longer SV4.2
- net HALL5_IN: now also JP19.1; no longer SV2.5
- net HALL6: now also JP16.4; no longer SV4.4
- net HALL6_IN: now also JP19.2; no longer SV2.6
- net HALL7: now also JP16.6; no longer SV4.6
- net HALL7_IN: now also JP20.1; no longer SV2.7
- net HALL8: now also JP16.8; no longer SV4.8
- net HALL8_IN: now also JP20.2; no longer SV2.8
- net N$1: now also JP13.1; no longer SV5.1
- net N$15: now also JP13.6; no longer SV5.6
- net N$16: now also JP13.3; no longer SV5.3
- net N$2: now also JP13.2; no longer SV5.2
- net N$29: now also JP11.1; no longer SV7.1
- net N$30: now also JP11.2; no longer SV7.2
- net N$32: now also JP11.4; no longer SV7.4
- net N$33: now also JP11.5; no longer SV7.5
- net N$34: now also JP11.6; no longer SV7.6
- net N$35: now also JP11.3; no longer SV7.3
- net N$4: now also JP13.4; no longer SV5.4
- net N$42: now also JP14.1; no longer SV6.1
- net N$43: now also JP14.2; no longer SV6.2
- net N$45: now also JP14.4; no longer SV6.4
- net N$46: now also JP14.5; no longer SV6.5
- net N$47: now also JP14.6; no longer SV6.6
- net N$48: now also JP14.3; no longer SV6.3
- net N$58: now also JP12.1; no longer SV8.1
- net N$59: now also JP12.2; no longer SV8.2
- net N$61: now also JP12.4; no longer SV8.4
- net N$62: now also JP12.5; no longer SV8.5
- net N$63: now also JP12.6; no longer SV8.6
- net N$64: now also JP12.3; no longer SV8.3
- net N$7: now also JP13.5; no longer SV5.5
- net N$77: now also JP15.13; no longer SV3.13
- net N$78: now also JP15.5; no longer SV3.5
- net N$79: now also JP15.6; no longer SV3.6
- net N$80: now also JP15.14; no longer SV3.14
